File: RFIDZapper.kicad_pcb (KiCad board)
At the start: 2 copper layers, 29 parts, among them Q1 BC549, Q2 P3NB90 FP, Q3 BC549, Q4 IRF9630G, U1 NE555, U2 L7805, U3 LM393

Commit message: Add files via upload
Parts:
- U1: footprint Housings_DIP:DIP-8_W7.62mm_Socket_LongPads -> Housings_DIP:DIP-8_W7.62mm_LongPads
- U3: value LM393 -> TL071; footprint Housings_DIP:DIP-8_W7.62mm_Socket_LongPads -> Housings_DIP:DIP-8_W7.62mm_LongPads
- moved C2 24.7 mm to (164.1, 93.2), turned to 180 degrees
- moved L1 17.3 mm to (145.3, 98.6), turned to 270 degrees
- moved Q2 15.0 mm to (178.6, 42.4)
- moved D3 14.9 mm to (155.4, 93.2), turned to 180 degrees
- moved SW_SPST3 14.0 mm to (158.2, 101.1)
- moved D1 12.2 mm to (165.1, 42.4)
- moved AE1 11.0 mm to (168.4, 112.3)
- moved R4 7.62 mm to (167.1, 73.4), turned to 180 degrees
- moved R5 7.62 mm to (159.5, 81.0), turned to 0 degrees
- moved R7 7.62 mm to (145.3, 67.8), turned to 0 degrees
- moved Q1 2.79 mm to (177.5, 86.9), turned to 0 degrees
- moved D2 2.30 mm to (150.1, 54.9), turned to 180 degrees
- moved C3 1.93 mm to (153.7, 117.1)
- moved R6 1.52 mm to (152.9, 59.4)
- moved U1 0.25 mm to (186.7, 81.0)
Connections:
- SW_SPST1 pad 1: /VDD -> /VCC
- SW_SPST1 pad 2: /VCC -> /VDD
- U3 pad 1: Net-(Q3-Pad2) -> Net-(U3-Pad1)
- U3 pad 5: (no net) -> Net-(U3-Pad5)
- U3 pad 6: (no net) -> Net-(Q3-Pad2)
- U3 pad 7: (no net) -> /VDD
- U3 pad 8: /VDD -> Net-(U3-Pad8)
Routing:
- net GNDPWR: track 147.8 -> 17.2 mm
- net Net-(AE1-Pad1): track 67.4 -> 10.2 mm
- net A: track 53.4 -> 108.6 mm
- net Net-(C2-Pad1): track 113.4 -> 146.3 mm
- net Net-(D3-Pad2): track 67.6 -> 96.0 mm
- net C: track 24.9 -> 47.9 mm
- net Net-(D1-Pad1): track 98.9 -> 82.2 mm
- net Net-(Q3-Pad2): track 51.4 -> 36.3 mm
- net Net-(D1-Pad3): track 28.4 -> 15.8 mm
- net Net-(Q3-Pad1): track 53.7 -> 60.7 mm
- net /VDD: track 154.6 -> 148.7 mm
- net Net-(C3-Pad1): track 49.6 -> 44.0 mm
- net Net-(D2-Pad2): track 9.58 -> 5.52 mm
- net Net-(Q1-Pad2): track 10.7 -> 10.1 mm
- added copper zone on B.Cu, net (none)
- added copper zone on B.Cu, net GNDPWR
