File: RFIDZapper.sch (KiCad schematic (older format))
At the start: 29 parts, among them Q1 BC549, Q2 P3NB90 FP, Q3 BC549, Q4 IRF9630G, U1 NE555, U2 L7805, U3 LM393

Commit message: Add files via upload
Parts:
- removed U3: LM393, Housings_DIP:DIP-8_W7.62mm_Socket_LongPads, symbol LM393
- added U3: TL071, Housings_DIP:DIP-8_W7.62mm_LongPads, symbol TL071
- U1: footprint Housings_DIP:DIP-8_W7.62mm_Socket_LongPads -> Housings_DIP:DIP-8_W7.62mm_LongPads
Connections:
- net B: now also U3.2 (-)
- net GNDPWR: now also U3.4 (V-)
- net VDD: now also U3.7 (V+)
- net at C2.1, R5.1, U2.3 (OUT): now also U3.3 (+)
- net at Q3.2 (B), R7.2: now also U3.6
- no-connect marks 1 -> 3
Changed lines of the file:
@@
-$EndComp
-$Comp
-L LM393 U3
-U 1 1 59B61200
-P 7800 1700
-F 0 "U3" H 8141 1746 50  0000 L CNN
-F 1 "LM393" H 8141 1655 50  0000 L CNN
-F 2 "Housings_DIP:DIP-8_W7.62mm_Socket_LongPads" H 7800 1700 50  0001 C CNN
-F 3 "" H 7800 1700 50  0001 C CNN
-	1    7800 1700
-	1    0    0    -1
 $EndComp
 $Comp
@@
 F 0 "U1" H 2050 2978 50  0000 C CNN
 F 1 "NE555" H 2050 2887 50  0000 C CNN
-F 2 "Housings_DIP:DIP-8_W7.62mm_Socket_LongPads" H 2050 2400 50  0001 C CNN
+F 2 "Housings_DIP:DIP-8_W7.62mm_LongPads" H 2050 2400 50  0001 C CNN
 F 3 "" H 2050 2400 50  0001 C CNN
 	1    2050 2400
@@
 Text Label 6800 1550 0    60   ~ 0
 5v
+$Comp
+L TL071 U3
+U 1 1 59B75E66
+P 7800 1700
+F 0 "U3" H 8141 1746 50  0000 L CNN
+F 1 "TL071" H 8141 1655 50  0000 L CNN
+F 2 "Housings_DIP:DIP-8_W7.62mm_LongPads" H 7850 1750 50  0001 C CNN
+F 3 "" H 7950 1850 50  0001 C CNN
+	1    7800 1700
+	1    0    0    -1
+$EndComp
+NoConn ~ 7800 2000
+NoConn ~ 7900 2000
 $EndSCHEMATC
