File: project/RFIDZapper.sch (KiCad schematic (older format))
At the start: 29 parts, among them Q1 BC549, Q2 P3NB90 FP, Q3 BC549, Q4 IRF9630G, U1 NE555, U2 L7805, U3 TL071

Commit message: Better 3D
Parts:
- R2: footprint Potentiometers:Potentiometer_Trimmer_Bourns_3266Y -> Potentiometers:Potentiometer_Trimmer_Bourns_3296W
Connections:
- net C: now also D1.1 (A1), L1.1, R6.1; no longer D1.2 (A2), Q4.2 (D)
- net A: no longer names the net of Q1.1 (C), Q2.1 (G), R4.2
- new net: D1.2 (A2), Q4.2 (D)
Other:
- moved on the sheet: AE1, BT1, C1, C2, C3, D1, D2, D3, L1, Q1, Q2, Q3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
