File: project-lite/RFIDZapper.sch (KiCad schematic (older format))
At the start: 22 parts, among them Q1 BC549, Q2 P3NB90 FP, U1 NE555

Commit message: Minor fixes
Connections:
- net VHI: now reaches C3.1, D3.1 (K), R8.1, SW_SPST3.1 (A)
- net OUT renamed PWM
- net VDD renamed VLO
Other:
- moved on the sheet: BT1, C1, C3, DL1, DZ1, Q1, R6, R8, R9
