File: project-lite/RFIDZapper.kicad_pcb (KiCad board)
At the start: 2 copper layers, 22 parts, among them Q1 BC549, Q2 P3NB90 FP, U1 NE555

Commit message: Lite routed
Parts:
- added G***: LOGO, Graphics:open-source-hardware_5mm, F.Cu at (157.6, 126.3)
- added G***: LOGO, Graphics:rfidzapper_5mm, F.Cu at (121.4, 126.1)
- added G***: LOGO, Graphics:high-voltaje_5mm, F.Cu at (114.4, 126.1)
- added G***: LOGO, Graphics:gitqrcode_5mm, F.Cu at (151.4, 126.3)
- AE1: footprint RF_Modules:NFC_ANTENNA2 -> RF_Modules:NFC_ANTENNA2_INSIDE_CONNECTION
- moved BT1 84.7 mm to (115.4, 113.8), turned to 270 degrees
- moved DZ1 77.5 mm to (148.6, 101.8)
- moved R9 75.5 mm to (148.6, 95.3)
- moved C1 74.1 mm to (158.4, 119.6), turned to 180 degrees
- moved C3 70.8 mm to (125.6, 93.3), turned to 0 degrees
- moved AE1 68.1 mm to (107.1, 104.8)
- moved L1 67.1 mm to (153.1, 95.8)
- moved Q2 67.0 mm to (155.9, 91.6)
- moved C2 66.9 mm to (134.6, 119.6)
- moved D1 66.9 mm to (148.9, 110.8)
- moved D2 66.9 mm to (141.4, 115.8)
- moved R1 66.9 mm to (141.4, 106.8)
- moved R3 66.9 mm to (141.4, 120.3)
- moved U1 66.9 mm to (128.4, 107.3)
- moved Q1 66.7 mm to (123.1, 113.3)
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Routing:
- net GNDPWR: track 0.00 -> 104.1 mm
- net /VDD: track 0.00 -> 74.1 mm
- net OUT: track 9.65 -> 68.2 mm
- net Net-(DL1-Pad2): track 0.00 -> 41.6 mm
- net /THR: track 8.67 -> 47.6 mm
- net Net-(C3-Pad1): track 4.50 -> 38.4 mm
- net Net-(DZ1-Pad2): track 0.00 -> 30.1 mm
- net Net-(D3-Pad2): track 0.00 -> 21.3 mm
- net Net-(DZ1-Pad1): track 0.00 -> 12.7 mm
- net Net-(R2-Pad1): track 0.00 -> 11.3 mm
- net Net-(AE1-Pad1): track 0.00 -> 8.93 mm
- net /VCC: track 0.00 -> 7.92 mm
- net Net-(R1-Pad2): track 0.00 -> 7.88 mm
- net RST: track 11.6 -> 12.9 mm
- added copper zone on B.Cu, net (none)
Other:
- net class Default: trace_width 1 -> 0.25
- board text added: "CERN Licence v1.2"
- board text added: "http://git.io/v5DJb"

Commit message: Add files via upload
Routing:
- net GNDPWR: track 104.1 -> 110.0 mm
- net OUT: track 68.2 -> 67.3 mm
Other:
- net class Default: trace_width 0.25 -> 1
- board text added: "WARNING! High Voltage!"
Changed lines of the file:
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@@
   (general
     (thickness 1.6)
-    (drawings 2)
-    (tracks 150)
+    (drawings 3)
+    (tracks 156)
     (zones 0)
     (modules 26)
@@
   )
   (setup
-    (last_trace_width 0.25)
+    (last_trace_width 1)
     (trace_clearance 0.5)
     (zone_clearance 0.508)
@@
     (visible_elements FFFFFF7F)
     (pcbplotparams
-      (layerselection 0x00030_ffffffff)
+      (layerselection 0x000f0_ffffffff)
       (usegerberextensions false)
       (usegerberattributes true)
@@
   (net_class Default "This is the default net class."
     (clearance 0.5)
-    (trace_width 0.25)
+    (trace_width 1)
     (via_dia 0.8)
     (via_drill 0.4)
@@
       (xy -2.629647 1.344706) (xy -2.629647 1.135529) (xy -1.165412 1.135529) (xy -1.165412 2.599765)) (layer F.SilkS) (width 0.01))
   )
+  (gr_text "WARNING! High Voltage!" (at 137.394 82.556) (layer F.SilkS)
+    (effects (font (size 1.5 1.5) (thickness 0.3)))
+  )
   (gr_text "CERN Licence v1.2" (at 135.894 127.806) (layer F.SilkS)
     (effects (font (size 1.5 1.5) (thickness 0.3)))
@@
   (segment (start 111.644 99.306) (end 115.394 95.556) (width 1) (layer B.Cu) (net 1))
   (segment (start 115.394 95.556) (end 115.394 92.886) (width 1) (layer B.Cu) (net 1) (status 800000))
+  (segment (start 158.394 119.556) (end 154.393998 123.556002) (width 1) (layer B.Cu) (net 2) (status 400000))
+  (segment (start 154.393998 123.556002) (end 154.144002 123.556002) (width 1) (layer B.Cu) (net 2))
+  (segment (start 154.144002 123.556002) (end 154.144 123.556) (width 1) (layer B.Cu) (net 2))
+  (segment (start 154.144 123.556) (end 154.144 123.556002) (width 1) (layer B.Cu) (net 2))
   (segment (start 123.144 110.766) (end 123.184 110.766) (width 1) (layer B.Cu) (net 2) (status C00000))
   (segment (start 129.644 119.556) (end 129.394 119.556) (width 1) (layer B.Cu) (net 2) (status C00000))
@@
   (segment (start 160.144 121.306) (end 160.144 122.556) (width 1) (layer B.Cu) (net 2))
   (segment (start 160.144 122.556) (end 159.143998 123.556002) (width 1) (layer B.Cu) (net 2))
-  (segment (start 159.143998 123.556002) (end 125.393998 123.556002) (width 1) (layer B.Cu) (net 2))
+  (segment (start 159.143998 123.556002) (end 154.144 123.556002) (width 1) (layer B.Cu) (net 2))
+  (segment (start 154.144 123.556002) (end 125.393998 123.556002) (width 1) (layer B.Cu) (net 2))
   (segment (start 125.393998 123.556002) (end 120.144002 123.556002) (width 1) (layer B.Cu) (net 2))
   (segment (start 141.144 91.056) (end 141.144 87.056) (width 1) (layer B.Cu) (net 3) (status C00000))
@@
   (segment (start 148.644 95.306) (end 148.644 91.176) (width 1) (layer B.Cu) (net 15) (status C00000))
   (segment (start 148.644 91.176) (end 148.764 91.056) (width 1) (layer B.Cu) (net 15) (status C00000))
+  (segment (start 157.519 117.681) (end 155.144 120.056) (width 1) (layer B.Cu) (net 16))
+  (segment (start 155.144 120.056) (end 155.144 120.556) (width 1) (layer B.Cu) (net 16))
+  (segment (start 155.144 120.556) (end 153.644 122.056) (width 1) (layer B.Cu) (net 16))
   (segment (start 159.144 116.056) (end 159.144 107.556) (width 1) (layer B.Cu) (net 16))
   (segment (start 159.144 107.556) (end 158.394 106.806) (width 1) (layer B.Cu) (net 16))
-  (segment (start 152.644 122.056) (end 155.144 122.056) (width 1) (layer B.Cu) (net 16))
-  (segment (start 155.144 122.056) (end 156.394 120.806) (width 1) (layer B.Cu) (net 16))
-  (segment (start 156.394 120.806) (end 156.394 118.806) (width 1) (layer B.Cu) (net 16))
-  (segment (start 156.394 118.806) (end 159.144 116.056) (width 1) (layer B.Cu) (net 16))
+  (segment (start 152.644 122.056) (end 153.644 122.056) (width 1) (layer B.Cu) (net 16))
+  (segment (start 157.519 117.681) (end 159.144 116.056) (width 1) (layer B.Cu) (net 16))
   (segment (start 155.894 91.556) (end 155.894 104.306) (width 1) (layer B.Cu) (net 16) (status 400000))
   (segment (start 155.894 104.306) (end 158.394 106.806) (width 1) (layer B.Cu) (net 16))

Commit message: New Lite
Parts:
- moved C3 32.0 mm to (157.6, 94.6), turned to 180 degrees
- moved L1 22.0 mm to (132.4, 103.1), turned to 0 degrees
- moved Q2 21.0 mm to (134.9, 90.8), turned to 0 degrees
- moved R6 19.8 mm to (129.4, 103.6)
- moved DZ1 19.4 mm to (129.4, 99.8)
- moved R9 19.3 mm to (129.4, 95.8)
- moved D3 19.2 mm to (121.9, 88.1)
- moved R8 19.2 mm to (121.9, 92.1)
- moved Q1 4.12 mm to (122.1, 109.3), turned to 0 degrees
- moved DL1 0.79 mm to (124.6, 118.8)
- moved AE1 0.25 mm to (106.9, 104.8)
Routing:
- net GNDPWR: track 110.0 -> 10.7 mm
- net OUT: track 67.3 -> 94.4 mm
- net Net-(DL1-Pad2): track 41.6 -> 16.7 mm
- net /VDD: track 74.1 -> 52.1 mm
- net Net-(DZ1-Pad2): track 30.1 -> 9.51 mm
- net Net-(C3-Pad1): track 38.4 -> 55.5 mm
- net Net-(D3-Pad2): track 21.3 -> 16.6 mm
- net Net-(DZ1-Pad1): track 12.7 -> 8.23 mm
- net RST: track 12.9 -> 14.8 mm
- net Net-(AE1-Pad1): track 8.93 -> 9.74 mm
- removed copper zone on B.Cu, net (none)

Commit message: Cap rotated
Parts:
- moved C3 5.48 mm to (153.6, 90.8), turned to 270 degrees
Routing:
- net Net-(C3-Pad1): track 55.5 -> 46.6 mm
Changed lines of the file:
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@@
   )
   (module Capacitors_ThroughHole:CP_Radial_D18.0mm_P7.50mm (layer F.Cu)
-    (at 157.644 94.556 180)
+    (at 153.644 90.806 270)
     (descr "CP, Radial series, Radial, pin pitch=7.50mm, , diameter=18mm, Electrolytic Capacitor")
     (tags "CP Radial series Radial pin pitch 7.50mm  diameter 18mm Electrolytic Capacitor")
-    (fp_text reference C3 (at 0 -3.81 180) (layer F.SilkS)
-      (effects (font (size 1 1) (thickness 0.15)))
-    )
-    (fp_text value "120uF 400v" (at 3.048 0 -90) (layer F.Fab)
-      (effects (font (size 1 1) (thickness 0.15)))
-    )
-    (fp_text user %R (at 0 -3.81 180) (layer F.Fab)
+    (fp_text reference C3 (at 0 -3.81 270) (layer F.SilkS)
+      (effects (font (size 1 1) (thickness 0.15)))
+    )
+    (fp_text value "120uF 400v" (at 3.048 0) (layer F.Fab)
+      (effects (font (size 1 1) (thickness 0.15)))
+    )
+    (fp_text user %R (at 0 -3.81 270) (layer F.Fab)
       (effects (font (size 1 1) (thickness 0.15)))
     )
@@
     (fp_circle (center 3.75 0) (end 12.84 0) (layer F.SilkS) (width 0.12))
     (fp_circle (center 3.75 0) (end 12.75 0) (layer F.Fab) (width 0.1))
-    (pad 2 thru_hole circle (at 7.5 0 180) (size 2.4 2.4) (drill 1.2) (layers *.Cu *.Mask)
+    (pad 2 thru_hole circle (at 7.5 0 270) (size 2.4 2.4) (drill 1.2) (layers *.Cu *.Mask)
       (net 2 GNDPWR))
-    (pad 1 thru_hole rect (at 0 0 180) (size 2.4 2.4) (drill 1.2) (layers *.Cu *.Mask)
+    (pad 1 thru_hole rect (at 0 0 270) (size 2.4 2.4) (drill 1.2) (layers *.Cu *.Mask)
       (net 3 "Net-(C3-Pad1)"))
     (model ${KISYS3DMOD}/Capacitors_THT.3dshapes/CP_Radial_D18.0mm_P7.50mm.wrl
@@
   (segment (start 110.442 110.306) (end 111.894 110.306) (width 1) (layer B.Cu) (net 2) (status 400000))
   (segment (start 111.894 110.306) (end 111.192 110.306) (width 1) (layer B.Cu) (net 2) (status 800000))
-  (segment (start 157.644 94.556) (end 157.644 90.556) (width 1) (layer B.Cu) (net 3) (status 400000))
-  (segment (start 146.144 86.056) (end 154.894 86.056) (width 1) (layer B.Cu) (net 3))
-  (segment (start 154.894 86.056) (end 157.644 88.806) (width 1) (layer B.Cu) (net 3))
-  (segment (start 157.644 88.806) (end 157.644 90.556) (width 1) (layer B.Cu) (net 3))
-  (segment (start 157.644 90.556) (end 157.644 91.806) (width 1) (layer B.Cu) (net 3))
+  (segment (start 153.644 90.806) (end 153.644 88.556) (width 1) (layer B.Cu) (net 3) (status 400000))
+  (segment (start 153.644 88.556) (end 151.144 86.056) (width 1) (layer B.Cu) (net 3))
+  (segment (start 146.144 86.056) (end 151.144 86.056) (width 1) (layer B.Cu) (net 3))
   (segment (start 146.144 86.056) (end 145.894 86.056) (width 1) (layer B.Cu) (net 3))
   (segment (start 121.944 88.056) (end 121.944 87.756) (width 1) (layer B.Cu) (net 3) (status C00000))
@@
   (segment (start 129.564 95.636) (end 129.394 95.806) (width 1) (layer B.Cu) (net 15) (status C00000))
   (segment (start 129.444 92.176) (end 129.564 92.056) (width 1) (layer B.Cu) (net 15) (status C00000))
+  (segment (start 144.394 100.556) (end 147.894 104.056) (width 1) (layer B.Cu) (net 16))
+  (segment (start 147.894 104.056) (end 156.894 104.056) (width 1) (layer B.Cu) (net 16))
+  (segment (start 156.894 104.056) (end 158.019 105.181) (width 1) (layer B.Cu) (net 16))
   (segment (start 134.894 98.306) (end 134.894 99.056) (width 1) (layer B.Cu) (net 16))
   (segment (start 134.894 99.056) (end 136.394 100.556) (width 1) (layer B.Cu) (net 16))
@@
   (segment (start 134.894 98.306) (end 134.894 99.056) (width 1) (layer B.Cu) (net 16))
   (segment (start 134.894 99.056) (end 136.394 100.556) (width 1) (layer B.Cu) (net 16))
-  (segment (start 158.019 105.181) (end 153.394 100.556) (width 1) (layer B.Cu) (net 16))
-  (segment (start 153.394 100.556) (end 136.394 100.556) (width 1) (layer B.Cu) (net 16))
+  (segment (start 144.394 100.556) (end 136.394 100.556) (width 1) (layer B.Cu) (net 16))
   (segment (start 158.019 105.181) (end 159.144 106.306) (width 1) (layer B.Cu) (net 16))
   (segment (start 128.394 112.386) (end 130.974 112.386) (width 1) (layer B.Cu) (net 16) (status 400000))

Commit message: Minor fixes
Parts:
- moved AE1 50.4 mm to (65.1, 133.1)
- moved BT1 50.4 mm to (73.6, 142.1)
- moved C1 50.4 mm to (116.6, 147.8)
- moved C2 50.4 mm to (92.9, 147.8)
- moved C3 50.4 mm to (111.9, 119.1)
- moved D1 50.4 mm to (107.1, 139.1)
- moved D2 50.4 mm to (99.6, 144.1)
- moved D3 50.4 mm to (80.2, 116.3)
- moved DL1 50.4 mm to (82.9, 147.1)
- moved DZ1 50.4 mm to (87.6, 128.1)
- moved G*** 50.4 mm to (115.9, 154.6)
- moved G*** 50.4 mm to (79.6, 154.3)
- moved G*** 50.4 mm to (72.6, 154.3)
- moved G*** 50.4 mm to (109.6, 154.6)
- moved L1 50.4 mm to (90.6, 131.3)
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Connections:
- net /VDD renamed /VLO
- net Net-(C3-Pad1) renamed /VHI
- net OUT renamed PWM
Other:
- net class Default: trace_width 1 -> 0.25
